File: hardware/smartbag_core.kicad_sch (KiCad schematic)
At the start: 26 parts, among them J1 FFC optics, 10 way, J2 LiPo 3.7V 2000mAh, J3 Qi RX coil, J4 FFC FSR matrix, 24 way, J5 SWD debug, U1 SoC+NPU BLE 5.4, U2 mmWave 60GHz TRX, U3 PMIC buck-boost, U4 6-axis IMU, U5 Hall, zip, Y1 32 MHz

Commit message: Rebuild the board around parts you can actually buy
The board was drawn from component classes with invented pinouts. It said
so, and it was still unbuildable. Every IC is now a real part whose pinout
comes from its own datasheet, and tools/bom_report.py measures each
footprint against the datasheet's package on every run: 18 of 18 agree.

Finding the real parts changed the architecture three times, and each
change had already been asked for by something else in this repo:

- rf/feed_loss.py priced a central 60 GHz transceiver's feed at 8.2 dB one
  way. The Acconeer A121's datasheet says the antenna is inside the package
  and "it is not possible to connect trace antenna" — so there are now TWO
  sensors, one on each end island, and no 60 GHz copper on the board at
  all. ANT_A1 and ANT_A2 are gone.
- thermal/budget.py asked for charge current to be a function of cell
  temperature. RT1 is a 10k NTC into an nPM1300, which does JEITA charging
  in hardware.
- firmware/test_sb_fsr.c measured both scan modes the old board could run:
  phantom taxels at 39% of a real press, or real ones 83% light. The rows
  now land on six transimpedance amplifiers and the columns on a 16:1
  multiplexer.

And one thing the parts took away: no BLE SoC in a QFN has an NPU and a
camera interface. The processor is an nRF54L15, a 128 MHz Cortex-M33, and
recognition has to run on it. Survivable only because the firmware already
waits 2 s for an object to settle.

91 parts, four layers, routed: 1683 tracks, 393 vias, 0 DRC violations, 0
footprint errors, schematic parity clean, 3 unconnected pads of 462. In1.Cu
carries zero tracks and stays a solid ground reference.

New machinery, each written because something went wrong without it:

- place.py — the floorplan is a hint; 91 hand-typed coordinates collided in
  28 places. It also knows nothing may sit on a flex tail, after a pass put
  a 24-way connector out over one and off the board edge.
- stitch.py — routing cuts the top pour into isla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
Parts:
- removed J2: LiPo 3.7V 2000mAh, Connector_JST:JST_SH_SM02B-SRSS-TB_1x02-1MP_P1.00mm_Horizontal, symbol smartbag:CONN_2
- removed J3: Qi RX coil, Connector_JST:JST_SH_SM02B-SRSS-TB_1x02-1MP_P1.00mm_Horizontal, symbol smartbag:CONN_2
- removed J5: SWD debug, Connector_JST:JST_SH_SM04B-SRSS-TB_1x04-1MP_P1.00mm_Horizontal, symbol smartbag:CONN_4
- removed U1: SoC+NPU BLE 5.4, Package_DFN_QFN:QFN-48-1EP_6x6mm_P0.4mm_EP4.6x4.6mm, symbol smartbag:SOC_NPU_48
- removed U2: mmWave 60GHz TRX, Package_DFN_QFN:QFN-40-1EP_5x5mm_P0.4mm_EP3.8x3.8mm, symbol smartbag:MMWAVE_40
- removed U3: PMIC buck-boost, Package_DFN_QFN:QFN-24-1EP_4x4mm_P0.5mm_EP2.8x2.8mm, symbol smartbag:PMIC_24
- removed U4: 6-axis IMU, Package_LGA:Bosch_LGA-14_3x2.5mm_P0.5mm, symbol smartbag:IMU_14
- removed U5: Hall, zip, Package_TO_SOT_SMD:SOT-23, symbol smartbag:HALL_3
- removed Y1: 32 MHz, Crystal:Crystal_SMD_3225-4Pin_3.2x2.5mm, symbol smartbag:XTAL_4
- added C11: 0.3p C0G, Capacitor_SMD:C_0402_1005Metric, symbol smartbag:C
- added C20, C21, C22, C23, C30, C31, C32, C33, C43, C44, C45, C46, C60: 1u X5R, Capacitor_SMD:C_0402_1005Metric, symbol smartbag:C
- added C24, C25, C34, C35: 8p NP0, Capacitor_SMD:C_0402_1005Metric, symbol smartbag:C
- added C40, C41, C42: 10u X5R 6.3V, Capacitor_SMD:C_0402_1005Metric, symbol smartbag:C
- added C50, C51, C52, C61, C62, C63: 100n X7R, Capacitor_SMD:C_0402_1005Metric, symbol smartbag:C
- added J2: LiPo 3.7V 2000mAh, Connector_JST:JST_SH_SM02B-SRSS-TB_1x02-1MP_P1.00mm_Horizontal, symbol smartbag:CONN2
- added J3: Qi RX coil, Connector_JST:JST_SH_SM02B-SRSS-TB_1x02-1MP_P1.00mm_Horizontal, symbol smartbag:CONN2
- added J5: SWD debug, Connector_JST:JST_SH_SM04B-SRSS-TB_1x04-1MP_P1.00mm_Horizontal, symbol smartbag:CONN4
- added L3, L4: 2.2u 1.2A, Inductor_SMD:L_0603_1608Metric, symbol smartbag:L
- added R10: 6.8k 1%, Resistor_SMD:R_0402_1005Metric, symbol smartbag:R
- added R11: 1.2k 1%, Resistor_SMD:R_0402_1005Metric, symbol smartbag:R
- added R12: 0R, Resistor_SMD:R_0402_1005Metric, symbol smartbag:R
- added R40, R41, R42, R43, R44, R45: 8.2k 1%, Resistor_SMD:R_0402_1005Metric, symbol smartbag:R
- added R5: 10k 1%, Resistor_SMD:R_0402_1005Metric, symbol smartbag:R
- added R6: 1k 1%, Resistor_SMD:R_0402_1005Metric, symbol smartbag:R
- added R60, R61, R62, R63, R64, R65, R66, R67, R68, R69, R70, R71, R72, R73, R74, R75: 100k 1%, Resistor_SMD:R_0402_1005Metric, symbol smartbag:R
- added R7, R8: 4.7k 1%, Resistor_SMD:R_0402_1005Metric, symbol smartbag:R
- added RT1: 10k NTC B3380, Resistor_SMD:R_0402_1005Metric, symbol smartbag:R
- added U1: nRF54L15-QFAA-R, Package_DFN_QFN:QFN-48-1EP_6x6mm_P0.4mm_EP4.6x4.6mm, symbol smartbag:NRF54L15
- added U2, U6: Acconeer A121, SmartBag:Acconeer_A121_fcCSP50, symbol smartbag:A121
- added U3: nPM1300-QEAA-R7, Package_DFN_QFN:QFN-32-1EP_5x5mm_P0.5mm_EP3.45x3.45mm, symbol smartbag:NPM1300
- added U4: BMI270, Package_LGA:Bosch_LGA-14_3x2.5mm_P0.5mm, symbol smartbag:BMI270
- added U5: DRV5032FBDBZR, Package_TO_SOT_SMD:SOT-23, symbol smartbag:DRV5032
- added U7: CD74HC4067SM96, Package_SO:SSOP-24_5.3x8.2mm_P0.65mm, symbol smartbag:MUX16
- added U8, U9: TLV9064IPWR, Package_SO:TSSOP-14_4.4x5mm_P0.65mm, symbol smartbag:OPA_QUAD
- added Y1: 32 MHz Cl=8pF, Crystal:Crystal_SMD_2016-4Pin_2.0x1.6mm, symbol smartbag:XTAL4
- added Y2, Y3: 24 MHz, Crystal:Crystal_SMD_2016-4Pin_2.0x1.6mm, symbol smartbag:XTAL4
- AE1: value 2.4 GHz chip antenna -> 2450AT43F0100E
- C1, C2: value 100n -> 2.2u X6T 2.5V
- C3: value 4u7 -> 10u X6S 6.3V
- C4: value 1u -> 100n X7R
- C5: value 100n -> 2.2n X7R
- C6: value 10u -> 1.5p NP0
- C7, C8: value 22u -> 100n X7R
- L1: value 2u2 -> 4.7u 120mA
- L2: value 1u0 -> 2.7n; footprint Inductor_SMD:L_0603_1608Metric -> Inductor_SMD:L_0402_1005Metric
- R1, R2, R3: value 10k -> 10k 1%
- R4: value 100k -> 1M 1%
Connections:
- net CAM_CLK is gone; now on net SPI_SCK: J1.5 (SCK)
- net CAM_DATA is gone; now on net SPI_MOSI: J1.6 (MOSI)
- net TOF_INT is gone; now on net CAM_PWDN: J1.9 (PWDN)
- net BLE_ANT: now also L2.2, C11.1
- net CAM_PWDN: now also U1.1 (P1.00); no longer J1.7 (CAM_PWDN)
- net FSR_C0: now also R60.1, U7.9 (I0)
- net FSR_C1: now also R61.1, U7.8 (I1)
- net FSR_C10: now also R70.1, U7.21 (I10)
- net FSR_C11: now also R71.1, U7.20 (I11)
- net FSR_C12: now also R72.1, U7.19 (I12)
- net FSR_C13: now also R73.1, U7.18 (I13)
- net FSR_C14: now also R74.1, U7.17 (I14)
- net FSR_C15: now also R75.1, U7.16 (I15)
- net FSR_C2: now also R62.1, U7.7 (I2)
- net FSR_C3: now also R63.1, U7.6 (I3)
- net FSR_C4: now also R64.1, U7.5 (I4)
- net FSR_C5: now also R65.1, U7.4 (I5)
- net FSR_C6: now also R66.1, U7.3 (I6)
- net FSR_C7: now also R67.1, U7.2 (I7)
- net FSR_C8: now also R68.1, U7.23 (I8)
- net FSR_C9: now also R69.1, U7.22 (I9)
- net FSR_R0: now also R40.1, U8.2 (IN1-)
- net FSR_R1: now also R41.1, U8.6 (IN2-)
- net FSR_R2: now also R42.1, U8.9 (IN3-)
- net FSR_R3: now also R43.1, U8.13 (IN4-)
- net FSR_R4: now also R44.1, U9.2 (IN1-)
- net FSR_R5: now also R45.1, U9.6 (IN2-)
- net GND: now also R2.2, R3.2, C11.2, C20.2, C21.2, C22.2, C23.2, C24.2, C25.2, C30.2, C31.2, C32.2, C33.2, C34.2, C35.2, C40.2, C41.2, C42.2, C43.2, C44.2, C45.2, C46.2, C50.2, C51.2, C52.2, C60.2, C61.2, C62.2, C63.2, J2.2 (BAT-), J3.2 (BAT-), J5.4 (GND), R11.2, R12.2, R6.2, RT1.2, U1.32 (VSS_PA), U1.44 (VSS), U1.49 (EP), U2.A2, U2.A3 (GND), U2.A4 (GND), U2.A5 (GND), U2.A6 (GND), U2.A7 (GND), U2.A8 (GND), U2.A9, U2.B1, U2.B10, U2.B2 (GND), U2.B9 (GND), U2.C1 (GND), U2.C10 (GND), U2.D2 (GND), U2.D9 (GND), U2.E1 (GND), U2.E10, U2.E2 (GND), U2.E9 (GND), U2.F1, U2.F2 (GND), U2.F9 (GND), U2.G1 (GND), U2.G10 (GND), U2.H1, U2.H2 (GND), U2.H9 (GND), U2.J3 (GND), U2.J5 (GND), U2.J6 (GND), U2.J8 (GND), U2.K4 (GND), U2.K5, U2.K7 (GND), U3.10 (GPIO3), U3.11 (GPIO4), U3.2 (PVSS1), U3.23 (CC1), U3.24 (CC2), U3.26 (LED1), U3.27 (LED2), U3.30 (LSIN2), U3.31 (LSOUT2), U3.33 (EP), U3.6 (PVSS2), U3.8 (GPIO1), U3.9 (GPIO2), U4.1 (SDO), U4.10 (OCSB), U4.11 (OSDO), U4.2 (ASDx), U4.3 (ASCx), U4.6 (GNDIO), U4.7 (GND), U5.3 (GND), U6.A2, U6.A3 (GND), U6.A4 (GND), U6.A5 (GND), U6.A6 (GND), U6.A7 (GND), U6.A8 (GND), U6.A9, U6.B1, U6.B10, U6.B2 (GND), U6.B9 (GND), U6.C1 (GND), U6.C10 (GND), U6.D2 (GND), U6.D9 (GND), U6.E1 (GND), U6.E10, U6.E2 (GND), U6.E9 (GND), U6.F1, U6.F2 (GND), U6.F9 (GND), U6.G1 (GND), U6.G10 (GND), U6.H1, U6.H2 (GND), U6.H9 (GND), U6.J3 (GND), U6.J5 (GND), U6.J6 (GND), U6.J8 (GND), U6.K4 (GND), U6.K5, U6.K7 (GND), U7.12 (GND), U8.11 (V-), U9.11 (V-), Y1.2 (GND), Y1.4 (GND), Y2.2 (GND), Y2.4 (GND), Y3.2 (GND), Y3.4 (GND); no longer J1.10 (GND), R4.2
- net I2C_SCL: now also R8.1, U1.24 (P0.01), U3.14 (SCL), U4.13 (SCX); no longer R3.1
- net I2C_SDA: now also R7.1, U1.23 (P0.00), U3.13 (SDA), U4.14 (SDX); no longer R2.1
- net SPI_MISO: now also J1.7 (MISO), U1.15 (P2.04/SDI), U2.K3 (SPI_MISO), U6.K3 (SPI_MISO)
- net SPI_MOSI: now also U1.13 (P2.02/SDO), U2.K6 (SPI_MOSI), U6.K6 (SPI_MOSI)
- net SPI_SCK: now also U1.12 (P2.01/SCK), U2.K2 (SPI_CLK), U6.K2 (SPI_CLK)
- net SW1: now also L3.1, U3.3 (SW1); no longer L1.1
- net SW2: now also L4.1, U3.5 (SW2); no longer L2.1
- net SWDIO: now also J5.3 (SWDIO), U1.25 (SWDIO)
- net VBAT: now also C43.1, J2.1 (BAT+), U3.19 (VBAT); no longer C6.1
- net VDD_1V8: now also C20.1, C21.1, C22.1, C30.1, C31.1, C32.1, C41.1, L3.2, U2.C2 (VRX), U2.C9 (VTX), U2.D1 (VRX), U2.D10 (VTX), U2.J9 (VDIG), U3.1 (VOUT1), U6.C2 (VRX), U6.C9 (VTX), U6.D1 (VRX), U6.D10 (VTX), U6.J9 (VDIG); no longer C1.1, C3.1, C5.1, C8.1, L2.2
- net VDD_3V3: now also C3.1, C8.1, C23.1, C33.1, C42.1, C50.1, C51.1, C52.1, C61.1, C62.1, C63.1, J5.1 (VDD), L4.2, R10.1, R5.2, R7.2, R8.2, U1.10 (VDD), U1.22 (VDD), U1.36 (VDD), U1.47 (VDD), U1.48 (VDD), U2.J1 (RESET_N), U2.K9 (VIO), U3.12 (VDDIO), U3.32 (VOUT2), U4.12 (CSB), U4.5 (VDDIO), U4.8 (VDD), U5.1 (VCC), U6.J1 (RESET_N), U6.K9 (VIO), U7.24 (VCC), U8.4 (V+), U9.4 (V+); no longer C2.1, J1.2 (VDD), R1.2, R2.2, R3.2
- net VQI: now also C44.1, J3.1 (BAT+), U3.21 (VBUS)
- net LED_PWM renamed CS_CAM
- net CS_CAM: now also U1.17 (P2.06)
- net VBAT_SNS renamed SHPHLD
- net SHPHLD: now also U3.15 (SHPHLD)
- net nRESET renamed VSYS
- net VSYS: now also R4.2, C40.1, U3.20 (VSYS), U3.28 (LSIN1), U3.4 (PVDD)
- new net ADC0: R40.2, U1.5 (P1.04/AIN0), U8.1 (OUT1)
- new net ADC1: R41.2, U1.6 (P1.05/AIN1), U8.7 (OUT2)
- new net ADC2: R42.2, U1.7 (P1.06/AIN2), U8.8 (OUT3)
- new net ADC3: R43.2, U1.8 (P1.07/AIN3), U8.14 (OUT4)
- new net ADC4: R44.2, U1.39 (P1.11/AIN4), U9.1 (OUT1)
- new net ADC5: R45.2, U1.40 (P1.12/AIN5), U9.7 (OUT2)
- new net ANT_FEED: C6.1, L2.1, U1.31 (ANT)
- new net CAM_RESET: J1.10 (RST), U1.2 (P1.01)
- new net CS_RADAR_L: U1.14 (P2.03), U2.J2 (SPI_SS)
- new net CS_RADAR_R: U1.16 (P2.05/CSN), U6.J2 (SPI_SS)
- new net DCC: L1.1, U1.46 (DCC)
- new net DECA: C1.1, U1.43 (DECA)
- new net DECD: C2.1, U1.45 (DECD)
- new net DECRF: C5.1, U1.33 (DECRF)
- new net FSR_SINK: R12.1, U7.1 (COM)
- new net HALL_OUT: U1.28 (P0.03), U5.2 (OUT)
- new net IMU_INT1: U1.27 (P0.02), U4.4 (INT1)
- new net LED0: R6.1, U3.25 (LED0)
- new net MUX_EN_N: U1.21 (P2.10), U7.15 (EN)
- new net MUX_S0: U1.3 (P1.02), U7.10 (S0)
- new net MUX_S1: U1.4 (P1.03), U7.11 (S1)
- new net MUX_S2: U1.9 (P1.08), U7.14 (S2)
- new net MUX_S3: U1.11 (P2.00), U7.13 (S3)
- new net NRESET: R5.1, U1.30 (nRESET)
- new net NTC: R1.2, RT1.1, U3.18 (NTC)
- new net OPA_SPARE3: U9.8 (OUT3), U9.9 (IN3-)
- new net OPA_SPARE4: U9.13 (IN4-), U9.14 (OUT4)
- new net PMIC_IRQ: U1.29 (P0.04), U3.7 (GPIO0)
- new net RADAR_EN: U1.18 (P2.07), U2.F10 (ENABLE), U6.F10 (ENABLE)
- new net RADAR_IRQ_L: U1.19 (P2.08), U2.K8 (INTERRUPT)
- new net RADAR_IRQ_R: U1.20 (P2.09), U6.K8 (INTERRUPT)
- new net SWDCLK: J5.2 (SWCLK), U1.26 (SWDCLK)
- new net VBUSOUT: C45.1, U3.22 (VBUSOUT)
- new net VDD_CAM: C46.1, J1.2 (VDD), U3.29 (LSOUT1)
- new net VREF: C60.1, R10.2, R11.1, R60.2, R61.2, R62.2, R63.2, R64.2, R65.2, R66.2, R67.2, R68.2, R69.2, R70.2, R71.2, R72.2, R73.2, R74.2, R75.2, U8.10 (IN3+), U8.12 (IN4+), U8.3 (IN1+), U8.5 (IN2+), U9.10 (IN3+), U9.12 (IN4+), U9.3 (IN1+), U9.5 (IN2+)
- new net VSET1: R2.1, U3.17 (VSET1)
- new net VSET2: R3.1, U3.16 (VSET2)
- new net X24L_1: C24.1, U2.J10 (XIN), Y2.1 (XI)
- new net X24L_2: C25.1, U2.H10 (XOUT), Y2.3 (XO)
- new net X24R_1: C34.1, U6.J10 (XIN), Y3.1 (XI)
- new net X24R_2: C35.1, U6.H10 (XOUT), Y3.3 (XO)
- new net XTAL32M_1: U1.34 (XC1), Y1.1 (XI)
- new net XTAL32M_2: U1.35 (XC2), Y1.3 (XO)
- no-connect marks 0 -> 5

Commit message: Choose the camera, cost the inference, and let the antenna datasheet win
Three things were still open. Each turned out to be answerable rather
than a matter of taste, and two of them found errors.

CAMERA. The SoC has no camera interface, so the module has to be SPI:
Arducam Mega 3MP NoIR (B0435), six wires, no IR-cut filter, 3.3 V,
56-136 mA. J1 was carrying I2C, a power-down and a reset that this part
does not have; those three ways now carry the thing the board was
actually missing — a way to switch the illuminators. thermal/budget.py
had been costing them at 0.6 W for a hundredth of a second since before
there was anything to switch them with. Q1 is that switch, with a gate
pull-down so they are dark while the processor is in reset.

The camera also freed XL1/XL2, which are now a 32.768 kHz crystal. The
app puts an age on every position it reports; the internal RC is
+/-500 ppm, which is 43 seconds a day, and a claim about a clock deserves
a clock.

NPU. ml/inference_budget.py counts the MACs by running a tensor through
the model in classify.py with hooks, reads the camera's SPI ceiling from
the chosen part and the deadlines from firmware/smartbag.h. 6.99 M MACs
a frame, 110-191 ms end to end against a 2000 ms settle window: it fits
by 10.5x at the pessimistic bound. The NPU was never needed at this model
size. The same arithmetic sets a limit nobody had written down: 320x240
RGB565 is 461 ms for a three-frame burst against a 400 ms capture
timeout, so the camera must be configured low.

ANTENNA. Reading the Johanson datasheet found three errors:
- terminal 2 was tied to GROUND and the terminal table says NC. It is a
  mechanical anchor; grounding it loads the radiator and no match
  recovers from that. It had been there since the first netlist, because
  a pad tied to ground is unremarkable in every check this project runs.
- the body was recorded as 3.2 x 1.6 mm and is 6.0 x 2.0.
- the ground plane ran straight under it. The datasheet calls for a
  7.0 x 2.2 m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
Parts:
- added Q1: SI2302CDS-T1-GE3, Package_TO_SOT_SMD:SOT-23, symbol smartbag:NMOS
- added R13: 100k 1%, Resistor_SMD:R_0402_1005Metric, symbol smartbag:R
- added Y4: 32.768 kHz Cl=9pF, Crystal:Crystal_SMD_2012-2Pin_2.0x1.2mm, symbol smartbag:XTAL2
Connections:
- net CS_CAM: now also J1.6 (CS); no longer J1.8 (CS)
- net GND: now also J1.10 (GND), J1.7 (GND), Q1.2 (S), R13.2; no longer AE1.2 (GND)
- net I2C_SCL: no longer J1.3 (SCL)
- net I2C_SDA: no longer J1.4 (SDA)
- net SPI_MISO: now also J1.5 (MISO); no longer J1.7 (MISO)
- net SPI_MOSI: now also J1.4 (MOSI); no longer J1.6 (MOSI)
- net SPI_SCK: now also J1.3 (SCK); no longer J1.5 (SCK)
- net VSYS: now also J1.8 (LED+)
- net IR_LED_EN: now reaches U1.37 (P1.09)
- net IR_LED_EN: now also Q1.1 (G), R13.1
- net CAM_PWDN renamed IR_LED_K
- net IR_LED_K: now also Q1.3 (D); no longer U1.1 (P1.00)
- net CAM_RESET renamed XTAL32K_2
- net XTAL32K_2: now also Y4.2 (XO); no longer J1.10 (RST)
- new net XTAL32K_1: U1.1 (P1.00/XL1), Y4.1 (XI)

Commit message: The ToF sensor the firmware always assumed, and fiducials
Two production blockers, both of them things that were invisible to every
check this project runs.

THE TIME-OF-FLIGHT SENSOR. firmware/smartbag.h has declared
SB_EV_TOF_CROSSED since the first commit — the beam across the mouth
breaking is what arms the camera — dimensions.py has placed a sensor at
TOF_X = 48, and the films show it working. No schematic ever contained
one. The wake-up chain depended on an event no hardware could raise.

It is a VL53L1X (LGA-12, 4.9 x 2.5 mm, I2C, XSHUT and GPIO1), it lives on
the optics flex because it has to look across the opening, and J1 grew
from ten ways to twelve to carry its I2C, shutdown and interrupt. KiCad
ships the footprint, so nothing was hand-drawn.

tools/check.py now reads the firmware's event enum against the netlist and
asserts that every event has a net that could produce it. The check was
negative-tested: removing TOF_INT makes it fail with "SB_EV_TOF_CROSSED
needs TOF_INT".

FIDUCIALS. The board had none, which means no assembly house would quote
it — a placement machine finds the board by looking at fiducials, and this
one has two 50-ball BGAs at 0.5 mm pitch. Three global in an L, so the
machine can tell which way round the board is, plus one local beside each
A121, because at 0.5 mm pitch a reference 90 mm away across a flex strip
that has just been through reflow is not a reference.

They are in the NETLIST, not just on the board: placed board-only they
produce five "extra footprint" parity warnings forever. Getting them to
match took two more corrections, both of which were DRC being right — a
fiducial's pad has an EMPTY number because it is a camera target and not
a connection, so the symbol has no pins either; and the footprint carries
exclude_from_bom, so the symbol has to say in_bom no.

ERC 0, DRC 0 errors, schematic parity clean, 4 unconnected pads.

Co-Authored-By: Claude Opus 5 <noreply@anthropic.com>
Parts:
- removed J1: FFC optics, 10 way, Connector_FFC-FPC:Hirose_FH12-10S-0.5SH_1x10-1MP_P0.50mm_Horizontal, symbol smartbag:FFC_10
- added FID1, FID2, FID3, FID4, FID5: fiducial, Fiducial:Fiducial_1mm_Mask2mm, symbol smartbag:FIDUCIAL
- added J1: FFC optics, 12 way, Connector_FFC-FPC:Hirose_FH12-12S-0.5SH_1x12-1MP_P0.50mm_Horizontal, symbol smartbag:FFC_12
Connections:
- net CS_CAM: now also J1.6 (CS)
- net GND: now also J1.1 (GND)
- net I2C_SCL: now also J1.8 (SCL)
- net I2C_SDA: now also J1.7 (SDA)
- net IR_LED_K: now also J1.12 (LED-)
- net SPI_MISO: now also J1.5 (MISO)
- net SPI_MOSI: now also J1.4 (MOSI)
- net SPI_SCK: now also J1.3 (SCK)
- net VDD_CAM: now also J1.2 (VDD)
- net VSYS: now also J1.11 (LED+)
- net TOF_XSHUT: now reaches U1.38 (P1.10)
- net TOF_XSHUT: now also J1.9 (XSHUT)
- net TOF_INT: now reaches U1.42 (P1.14/AIN7)
- net TOF_INT: now also J1.10 (TOF_INT)
- no-connect marks 5 -> 3

Commit message: Fiducials: the one part that can go anywhere, placed like it could not
Thirteen DRC violations on the routed board were all the same three parts.
A fiducial has no net, so nothing in the flow knew it was there: the
placement relaxer shoved two of them into capacitors and stalled, the
stitching via grid dropped a hole in a third, and freerouting ran a
VDD_3V3 track 0.44 mm from a fourth. A placement camera looking for a
round mark on bare soldermask would have found copper.

- fiducials are placed last, by search rather than by nudging, and their
  position is a decision the netlist states: two per rigid island,
  diagonally opposite, because the flex tails let the islands move with
  respect to each other. Maximising clearance instead — the first repair
  — emptied all of them onto the least crowded island and left three in
  a row, which tells a camera about one axis.
- a 2 mm keepout on every layer, which is the footprint's own soldermask
  opening, so the router and the pour both know. All three boards.
- the stitching grid applied its "is a part here?" test to one row out of
  five, and asked at the netlist's hint coordinates rather than where
  place.py had actually put things, up to 3.9 mm away.

Two more things fell out of chasing it:

- stitch.py chose via positions against the fill as it stood before the
  via existed, then refilled; an island narrow enough retracts away from
  the very via meant to anchor it, leaving a hole connected to nothing.
  It now checks its claim against the final fill and withdraws those.
  The optics flex goes 4 unconnected -> 1.
- the pipeline rebuilt the insert board from its routing session and
  regenerated the optics flex WITHOUT importing its own — so every run
  quietly reverted the flex to bare copper and then rendered it. The
  paragraph above that line argued for exactly the thing it did not do.

Also: generate_board.py could build the taxel sheet from its BOARDS
table, producing a legal board with none of the 1155 copp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
Parts:
- removed J2: LiPo 3.7V 2000mAh, Connector_JST:JST_SH_SM02B-SRSS-TB_1x02-1MP_P1.00mm_Horizontal, symbol smartbag:CONN2
- removed R1: 10k 1%, Resistor_SMD:R_0402_1005Metric, symbol smartbag:R
- removed RT1: 10k NTC B3380, Resistor_SMD:R_0402_1005Metric, symbol smartbag:R
- added C80: 270n C0G (Cs), Capacitor_SMD:C_0603_1608Metric, symbol smartbag:C
- added C81: 2n7 C0G (Cd), Capacitor_SMD:C_0402_1005Metric, symbol smartbag:C
- added C82, C83: 10n X7R, Capacitor_SMD:C_0402_1005Metric, symbol smartbag:C
- added C84, C85: 470n X7R 25V, Capacitor_SMD:C_0603_1608Metric, symbol smartbag:C
- added C86, C87: 47n X7R, Capacitor_SMD:C_0402_1005Metric, symbol smartbag:C
- added C88: 10u X5R 25V, Capacitor_SMD:C_0603_1608Metric, symbol smartbag:C
- added J2: LiPo 3.7V 2000mAh + NTC, Connector_JST:JST_SH_SM03B-SRSS-TB_1x03-1MP_P1.00mm_Horizontal, symbol smartbag:CONN3
- added R20: 220R 1%, Resistor_SMD:R_0402_1005Metric, symbol smartbag:R
- added R21: 100R 1%, Resistor_SMD:R_0402_1005Metric, symbol smartbag:R
- added R22: 10k 1%, Resistor_SMD:R_0402_1005Metric, symbol smartbag:R
- added U11: BQ51013BRHLR, Package_DFN_QFN:Texas_VQFN-RHL-20, symbol smartbag:BQ51013B
Connections:
- net GND: now also C88.2, J2.3 (BAT-), R21.2, R22.2, U11.1 (PGND), U11.10 (EN1), U11.11 (EN2), U11.20 (PGND), U11.21 (EP), U11.9 (AD); no longer J3.2 (BAT-)
- net NTC: now also J2.2 (NTC)
- net VBAT: now also J2.1 (BAT+)
- net VQI: now also U11.4 (OUT); no longer J3.1 (BAT+)
- new net QI_AC1: C80.2, C81.1, C82.2, C84.2, C86.2, U11.2 (AC1)
- new net QI_AC2: C81.2, C83.2, C85.2, C87.2, J3.2 (COIL_B), U11.19 (AC2)
- new net QI_BOOT1: C82.1, U11.3 (BOOT1)
- new net QI_BOOT2: C83.1, U11.17 (BOOT2)
- new net QI_CLAMP1: C84.1, U11.5 (CLAMP1)
- new net QI_CLAMP2: C85.1, U11.16 (CLAMP2)
- new net QI_COIL_A: C80.1, J3.1 (COIL_A)
- new net QI_COMM1: C86.1, U11.6 (COMM1)
- new net QI_COMM2: C87.1, U11.15 (COMM2)
- new net QI_FOD: R20.2, R21.1, U11.14 (FOD)
- new net QI_ILIM: R20.1, U11.12 (ILIM)
- new net QI_RECT: C88.1, U11.18 (RECT)
- new net QI_TS: R22.1, U11.13 (TS_CTRL)
- no-connect marks 3 -> 5

Commit message: Sixteen unconnected pads were a pin assignment, not a routing problem
The board came back from the router with one contiguous run of U1's pins
unrouted, and what they had in common was direction: every destination
was tens of millimetres east, and MUX_S3 sat on pin 11 — the west edge.
That net began by crossing the whole processor before it could start
travelling.

Which GPIO carries which signal is a layout decision, and on this part it
is nearly free: the firmware reaches pins through a HAL of symbolic ids,
so the physical assignment is invisible to it. The P2 block is now
ordered by destination — westbound nets on the west pins, eastbound on
the east, furthest travel outermost. SPI_SCK/MOSI/MISO do not move,
because those are the pins the high-speed SPIM is wired to in silicon and
the other instances run at 8 MHz instead of 32. CS_RADAR_R gives up
P2.05/CSN, which costs nothing: two radars share one bus, so at most one
chip select could ever have been the hardware CSN.

  unconnected     16 -> 4
  autoroute time  65 min -> 15 min
  DRC             0 errors, 0 footprint errors, parity clean

Four stitching vias were also outside the board. The rows at the ends run
along y = ±7.6, which is inside the 20 mm rigid islands and outside the
14 mm flex tails, and each row starts three millimetres into the tail.
DRC did not call them out-of-board; it called them unconnected, which is
the same fact told in a way that sounds like routing.

⛔ And a stale .pyc validated the bill of materials against a part number
that was no longer in the source. Restoring bom.py from a backup gave it
a size and timestamp matching the bytecode of the previous version, so
Python kept serving the old one and J2 passed as a 2-way connector for
several runs after being corrected to 3. Every number this project prints
comes from importing these files and measuring them, which makes that a
way to check the wrong file and be told it passed. The entry points now
set PYTHONDONTWRITEBYTECODE — writing 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
Parts:
- added FID6: fiducial, Fiducial:Fiducial_1mm_Mask2mm, symbol smartbag:FIDUCIAL
Connections:
- net CS_CAM: now also U1.16 (P2.05/CSN); no longer U1.17 (P2.06)
- net CS_RADAR_L: now also U1.11 (P2.00); no longer U1.14 (P2.03)
- net CS_RADAR_R: now also U1.21 (P2.10); no longer U1.16 (P2.05/CSN)
- net MUX_EN_N: now also U1.19 (P2.08); no longer U1.21 (P2.10)
- net MUX_S3: now also U1.18 (P2.07); no longer U1.11 (P2.00)
- net RADAR_EN: now also U1.17 (P2.06); no longer U1.18 (P2.07)
- net RADAR_IRQ_L: now also U1.14 (P2.03); no longer U1.19 (P2.08)
