File: hardware/smartbag_core.kicad_sch (KiCad schematic)
At the start: 111 parts, among them J1 FFC optics, 12 way, J2 Jauch LP523450JU 950mAh, J3 Qi RX coil, J4 FFC FSR matrix, 24 way, J5 SWD debug, Q1 SI2302CDS-T1-GE3, U1 nRF54L15-QFAA-R, U11 BQ51013BRHLR, U2 Acconeer A121, U3 nPM1300-QEAA-R7, U4 BMI270, U5 DRV5032FBDBZR, U6 Acconeer A121, U7 CD74HC4067SM96, U8 TLV9064IPWR, U9 TLV9064IPWR, Y1 32 MHz Cl=8pF, Y2 24 MHz, Y3 24 MHz, Y4 32.768 kHz Cl=9pF

Commit message: A bill of materials you can put in a basket
23 named parts, each with a manufacturer number whose package was
measured against its own datasheet — and none of that puts anything in a
cart. tools/order.py writes what a distributor takes: part number and
quantity, for a BUILD rather than for a board, because five prototypes of
a design with two radars on it is ten radars and the commonest way to be
short on assembly day is to have ordered one board's worth of something
that appears twice.

Trying to order found two parts that do not exist to order, the same way
the battery was found — by looking for a basket rather than for a
datasheet:

- U10 was "VL53L1X", which is the family. The orderable chip is
  VL53L1CXV0FY/1, $6.63.
- L_COIL was Würth 760308103305, which is not in Digi-Key's catalogue at
  all. 760308103202 is, and it fits the CAD exactly — 48 mm across, the
  24 mm radius cad/bag_and_insert.py has always drawn, 1.0 mm tall in a
  1.4 mm recess.

⛔ AND THE COIL CHANGED THE CIRCUIT. 12 µH instead of 8.8 moves both
resonant capacitors — Cs 270 → 220 nF, Cd 2.7 → 2.2 nF — and NOTHING
JOINED the calculation to the board. qi_resonance.py derived the values
and netlist.py had numbers typed into two capacitors; swapping the coil
would have left a tank tuned for a part nobody could buy, silently.
tools/check.py now compares the fitted values against the computation and
the BOM's coil against the one the computation used.

⚠️ Prices carry the date they were taken. $652.61 covers the twelve lines
that dominate the cost, at five boards; the fifteen left are 0402-class
commodity. A number in a repository does not go out of stock on its own,
which is why the deliverable is an upload file rather than a price list.

⚠️ And two lines decide the schedule rather than the cost: the coil showed
ZERO stock at Digi-Key, so it is the line to order first, and the cell is
a lithium pouch that ships under UN38.3 with couriers that may refuse it
by air.

The passives are a specificatio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
Parts:
- C80: value 270n C0G (Cs) -> 220n C0G (Cs)
- C81: value 2n7 C0G (Cd) -> 2n2 C0G (Cd)

Commit message: Forty-one of forty-one supply pins had no decoupling worth the name
The check did not exist, so I wrote it, and every IC supply pin on the board
failed it. The worst was the multiplexer at 26 mm — a 100 nF part twenty-six
millimetres from its pin is an inductor with a capacitor in series. The board
had been routed, DRC'd, rendered, costed and called orderable in that state.

And netlist.py said it was already fixed. "THE 100 nF PARTS HUG THE PINS THEY
DECOUPLE... the QFN has VDD on all four sides, so there is a capacitor on all
four sides", naming C5 as the one on the top edge — which is 2.2 nF on DECRF,
an internal regulator pin. U1 pins 47/48 never had decoupling and neither did
U7. A comment is not a check.

It could not not drift: place.py is a relaxation that only knows how to push
things apart. Nothing in it pulls anything toward anything, so every capacitor
walked away from its pin a third of a millimetre at a time. The intent moved
into a DECOUPLE map and the placer now reads the pin's real pad out of the
footprint and settles the capacitor against it after everything else.

Then the half that matters: C7 came back with its ground terminal on a 0.69 mm2
scrap of pour with no via in it. A capacitor 1 mm from its pin with a 20 mm
return is worse than one 3 mm away with a via underneath — the loop is both
sides. And it was caused by the first fix, because pressing capacitors against
packages is what pinches the pour off around them.

Then the escape channels. A QFN48 at 0.4 mm pitch escapes through a via ring
0.35 mm outside its pads and everything on that edge uses the gap; a 0402 in
the gap closes it. Measured: it cost RADAR_IRQ_R and CS_RADAR_R, two signals
that had routed for months. Widening the band the placer keeps clear got both
back. U1's own four are on the back, under their pins — which costs a second
assembly side and says so in the fab notes.

Four tool bugs fell out of it:

  - the relaxation pushed by a fixed step, so a part in a lane 1.82 mm tal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
Parts:
- added C64, C9: 100n X7R, Capacitor_SMD:C_0402_1005Metric, symbol smartbag:C
Connections:
- net GND: now also C64.2, C9.2
- net VDD_3V3: now also C64.1, C9.1
