File: hardware/smartbag_optics.kicad_pcb (KiCad board)
At the start: 2 copper layers, 134 x 12 mm, 15 parts, among them J10 FFC to insert, 12 way, J11 camera module, 6 way, U10 VL53L1X

Commit message: Fiducials: the one part that can go anywhere, placed like it could not
Thirteen DRC violations on the routed board were all the same three parts.
A fiducial has no net, so nothing in the flow knew it was there: the
placement relaxer shoved two of them into capacitors and stalled, the
stitching via grid dropped a hole in a third, and freerouting ran a
VDD_3V3 track 0.44 mm from a fourth. A placement camera looking for a
round mark on bare soldermask would have found copper.

- fiducials are placed last, by search rather than by nudging, and their
  position is a decision the netlist states: two per rigid island,
  diagonally opposite, because the flex tails let the islands move with
  respect to each other. Maximising clearance instead — the first repair
  — emptied all of them onto the least crowded island and left three in
  a row, which tells a camera about one axis.
- a 2 mm keepout on every layer, which is the footprint's own soldermask
  opening, so the router and the pour both know. All three boards.
- the stitching grid applied its "is a part here?" test to one row out of
  five, and asked at the netlist's hint coordinates rather than where
  place.py had actually put things, up to 3.9 mm away.

Two more things fell out of chasing it:

- stitch.py chose via positions against the fill as it stood before the
  via existed, then refilled; an island narrow enough retracts away from
  the very via meant to anchor it, leaving a hole connected to nothing.
  It now checks its claim against the final fill and withdraws those.
  The optics flex goes 4 unconnected -> 1.
- the pipeline rebuilt the insert board from its routing session and
  regenerated the optics flex WITHOUT importing its own — so every run
  quietly reverted the flex to bare copper and then rendered it. The
  paragraph above that line argued for exactly the thing it did not do.

Also: generate_board.py could build the taxel sheet from its BOARDS
table, producing a legal board with none of the 1155 copp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
Routing:
- net GND: vias 8 -> 7
